File: project files (kicad)/drone_esc_march_2026.kicad_pcb (KiCad board)
At the start: 4 copper layers, 77.8 x 108.6 mm, 180 parts, among them IC1 DRV8323RSRGZT, IC2 STM32F407VET6, IC3 DRV8323RSRGZT, IC4 DRV8323RSRGZT, IC5 DRV8323RSRGZT, J1 Screw_Terminal_01x03, J2 Screw_Terminal_01x03, J3 Screw_Terminal_01x03, J4 Screw_Terminal_01x03, Q1 MCG4D8N04YHE3-TP, Q10 MCG4D8N04YHE3-TP, Q11 MCG4D8N04YHE3-TP, Q12 MCG4D8N04YHE3-TP, Q13 MCG4D8N04YHE3-TP, Q14 MCG4D8N04YHE3-TP, Q15 MCG4D8N04YHE3-TP, Q16 MCG4D8N04YHE3-TP, Q17 MCG4D8N04YHE3-TP, Q18 MCG4D8N04YHE3-TP, Q19 MCG4D8N04YHE3-TP, Q2 MCG4D8N04YHE3-TP, Q20 MCG4D8N04YHE3-TP, Q21 MCG4D8N04YHE3-TP, Q22 MCG4D8N04YHE3-TP, Q23 MCG4D8N04YHE3-TP, Q24 MCG4D8N04YHE3-TP, Q25 IRF4905, Q3 MCG4D8N04YHE3-TP, Q4 MCG4D8N04YHE3-TP, Q5 MCG4D8N04YHE3-TP, Q6 MCG4D8N04YHE3-TP, Q7 MCG4D8N04YHE3-TP, Q8 MCG4D8N04YHE3-TP, Q9 MCG4D8N04YHE3-TP

Commit message: Update drone_esc_march_2026.kicad_pcb
Parts:
- moved R5 2.40 mm to (102.0, 108.9)
- moved R20 1.50 mm to (67.9, 54.3)
- moved R46 1.43 mm to (67.6, 115.7)
- moved R33 1.38 mm to (53.5, 68.9)
- moved C26 0.27 mm to (70.2, 58.5)
- moved C22 0.18 mm to (76.8, 62.0)
Routing:
- net SPI1_MISO: track 0.00 -> 143.9 mm, vias 0 -> 5
- net SPI1_MOSI: track 0.00 -> 140.1 mm, vias 0 -> 7
- net SPI1_SCK: track 0.00 -> 139.2 mm, vias 0 -> 6
- net EN_DRIVER_M2: track 0.00 -> 57.7 mm, vias 0 -> 2
- net SPI1_NSS_M2: track 0.00 -> 53.6 mm, vias 0 -> 2
- net lsideC_M3: track 0.00 -> 44.3 mm, vias 0 -> 2
- net lsideA_M3: track 0.00 -> 42.6 mm, vias 0 -> 2
- net hsideA_M3: track 0.00 -> 26.2 mm
- net hsideC_M3: track 0.00 -> 26.0 mm, vias 0 -> 2
- net hsideB_M3: track 0.00 -> 25.9 mm, vias 0 -> 2
- net hsideC_M4: track 0.00 -> 23.7 mm, vias 0 -> 2
- net lsideC_M4: track 0.00 -> 23.6 mm, vias 0 -> 2
- net Fault_M3: track 2.55 -> 24.3 mm
- net EN_DRIVER_M3: track 0.00 -> 21.7 mm
- net lsideA_M4: track 0.00 -> 20.4 mm, vias 0 -> 2
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
Commit message: Update drone_esc_march_2026.kicad_pcb
Updated some motor controller 2 traces to the central  controller
Parts:
- moved C43 1.10 mm to (65.2, 110.8)
- moved C10 0.61 mm to (98.5, 104.4)
Routing:
- net AMP_CALLIB: track 0.00 -> 114.0 mm, vias 0 -> 6
- net hsideA_M2: track 0.00 -> 50.3 mm, vias 0 -> 2
- net hsideB_M2: track 0.00 -> 49.3 mm, vias 0 -> 4
- net hsideC_M2: track 0.00 -> 47.2 mm, vias 0 -> 4
- net lsideC_M2: track 0.00 -> 24.6 mm, vias 0 -> 2
- net lsideA_M2: track 0.00 -> 24.2 mm, vias 0 -> 2
- net lsideB_M2: track 0.00 -> 23.9 mm, vias 0 -> 2
- net SPI1_MISO: track 143.9 -> 148.1 mm
- net EN_DRIVER_M2: track 57.7 -> 61.9 mm
- net SPI1_SCK: track 139.2 -> 142.0 mm
- net GND: track 322.2 -> 322.9 mm
